File: hw/oled_pcb/oled_board.kicad_pcb (KiCad board)
At the start: 4 copper layers, 35.4 x 9.1 mm, 14 parts, among them J19 Conn_01x01, J20 Conn_01x01, J21 Conn_01x01, J3 OLED

Commit message: 3d files and oled board
Parts:
- added J22: Conn_01x01, Connector_Wire:SolderWirePad_1x01_SMD_1x2mm, B.Cu at (167.2, 101.5)
- added TP1: TestPoint, TestPoint:TestPoint_Pad_D1.0mm, B.Cu at (169.0, 101.5)
- H1, H2: footprint MountingHole:MountingHole_2.2mm_M2_ISO7380 -> Mounting_Wuerth:Mounting_Wuerth_WA-SMSI-M2_H0.5mm_9774005243; moved to B.Cu
- moved C18 49.4 mm to (171.8, 107.2), turned to 0 degrees
- moved R12 48.1 mm to (174.9, 107.2)
- moved C14 48.1 mm to (171.8, 105.7)
- moved C16 47.3 mm to (175.0, 102.0), turned to 180 degrees
- moved J3 46.6 mm to (168.2, 104.6)
- moved H1 46.6 mm to (157.9, 104.5), turned to 180 degrees
- moved H2 46.6 mm to (189.0, 104.5), turned to 180 degrees
- moved C17 43.8 mm to (171.8, 102.0), turned to 180 degrees
- moved R13 43.5 mm to (171.8, 104.2)
- moved J19 43.4 mm to (165.7, 101.5), turned to 180 degrees
- moved J20 43.4 mm to (164.2, 101.5), turned to 180 degrees
- moved J21 43.4 mm to (162.7, 101.5)
- moved C22 42.7 mm to (167.2, 105.7), turned to -90 degrees
- moved C20 41.9 mm to (165.7, 105.7), turned to -90 degrees
Connections:
- J3 pad 7: unconnected-(J3-Pin_7-Pad7) -> GND
Routing:
- net Net-(J3-Pin_14): track 19.0 -> 4.82 mm
- net unconnected-(J3-Pin_7-Pad7): track 8.63 -> 0.00 mm
- net Net-(J3-Pin_13): track 14.3 -> 5.71 mm
- net Net-(J3-Pin_3): track 11.3 -> 3.99 mm
- net /DISP_VCC: track 23.9 -> 17.7 mm, vias 2 -> 1
- net /DISP_SCL: track 3.42 -> 7.16 mm
- net /DISP_SDA: track 5.13 -> 8.85 mm
- net Net-(J3-Pin_2): track 6.97 -> 10.2 mm
- net Net-(J3-Pin_12): track 14.1 -> 11.3 mm
- net /DISP_NRST: track 12.7 -> 10.6 mm
- net GND: track 0.00 -> 1.46 mm, vias 7 -> 32
- net Net-(J3-Pin_1): track 10.9 -> 9.64 mm
- net Net-(J3-Pin_4): track 6.80 -> 7.72 mm
- removed copper zone on In1.Cu, net GND
- removed copper zone on In2.Cu, net GND
Other:
- board size 35.4 x 9.1 mm -> 36.9 x 9.1 mm
- copper layers 4 -> 2
- board text added: "C"
- board text added: "D"
- board text added: "G"
- board text added: "R"
- board text added: "V"
