File: hw/oled_pcb/oled_board.kicad_sch (KiCad schematic)
At the start: 14 parts, among them J19 Conn_01x01, J20 Conn_01x01, J21 Conn_01x01, J3 OLED

Commit message: 3d files and oled board
Parts:
- added J22: Conn_01x01, Connector_Wire:SolderWirePad_1x01_SMD_1x2mm, symbol Connector_Generic:Conn_01x01
- added TP1: TestPoint, TestPoint:TestPoint_Pad_D1.0mm, symbol Connector:TestPoint
- H1, H2: footprint MountingHole:MountingHole_2.2mm_M2_ISO7380 -> Mounting_Wuerth:Mounting_Wuerth_WA-SMSI-M2_H0.5mm_9774005243; symbol Mechanical:MountingHole -> Mechanical:MountingHole_Pad
Connections:
- net DISP_NRST: now also TP1.1
- net GND: now also J3.7 (Pin_7), J22.1 (Pin_1)
- no-connect marks 1 -> 3
